File: bitClock.brd (EAGLE design)
At the start: 40 x 40 mm, 19 parts, among them U1 ATMEGA328P_TQFP

Commit message: new modification
Parts:
- added D19, D20, D21, D22, D23, D24, D25, D26, D27, D28, D29, D30, D31, D32, D33, D34, D35, D36, D37, D38, D39, D40, D41, D42, D43, D44, D45, D46, D47, D48, D49, D50, D51, D52, D53, D54, D55, D56, D57, D58, D59, D60: (no value), SparkFun-LED:LED-0603
- moved D11 32.9 mm to (8.24, 14.9), turned to 61 degrees
- moved D16 31.6 mm to (-0.45, 17.0), turned to 91.5 degrees
- moved D17 30.5 mm to (-2.26, 16.8), turned to 97.6 degrees
- moved D13 27.3 mm to (4.91, 16.3), turned to 73.2 degrees
- moved D5 26.6 mm to (15.5, 7.02), turned to 24.4 degrees
- moved D6 25.7 mm to (14.6, 8.63), turned to 30.5 degrees
- moved D7 24.9 mm to (13.6, 10.1), turned to 36.7 degrees
- moved D8 24.4 mm to (12.5, 11.5), turned to 42.7 degrees
- moved D10 24.4 mm to (9.77, 13.9), turned to 54.9 degrees
- moved D9 24.2 mm to (11.2, 12.8), turned to 48.8 degrees
- moved D14 21.7 mm to (3.15, 16.7), turned to 79.4 degrees
- moved D3 20.6 mm to (16.6, 3.59), turned to 12.2 degrees
- moved D1 20.6 mm to (17.0, 0.00), turned to 0 degrees
- moved D2 17.9 mm to (16.9, 1.81), turned to 6.1 degrees
- moved D18 16.7 mm to (-4.03, 16.5), turned to 103.7 degrees
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