File: bitClock.sch (EAGLE design)
At the start: 19 parts, among them U1 ATMEGA328P_TQFP

Commit message: new modification
Parts:
- added D19, D20, D21, D22, D23, D24, D25, D26, D27, D28, D29, D30, D31, D32, D33, D34, D35, D36, D37, D38, D39, D40, D41, D42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: (no value), SparkFun-LED:LED0603
Other:
- moved on the sheet: D1, D10, D11, D12, D13, D14, D15, D16, D17, D18, D2, D3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
